Commit message: WIP rae urdf model (#182)

File: depthai_bridge/urdf/rae.urdf.xacro (robot description, xacro)
@@ -5,5 +5,5 @@
       <inertial>
         <mass value="1.0"/>
-        <origin rpy="0 0 0" xyz="0 0 0"/>
+        <origin rpy="0.0 0.0 0.0" xyz="0.0 0.0 0.0"/>
         <inertia
           ixx = "0.166667"
@@ -22,14 +22,27 @@
       </collision>
       <visual>
-        <origin rpy="0.049227 0.011061 0.000747" xyz="-0 -1e-06 3.14159"/>
+        <origin rpy="0.0 0.0 0.0" xyz="0.0 0.0 0.0"/>
         <geometry>
           <mesh filename="package://depthai_bridge/urdf/models/rae_chassis.stl" scale="1.0 1.0 1.0"/>
         </geometry>
+        <material name="mat">
+          <lighting>1</lighting>
+          <!-- <color rgba="0.1 0.1 0.1 1.0"/> -->
+          <shader type='pixel'/>
+          <emissive>0 0 0 1</emissive>
+        </material>
+        <transparency>0</transparency>
+        <cast_shadows>1</cast_shadows>
       </visual>
     </link>
+    <joint name="base_chassis_joint" type="fixed">
+        <parent link="base_frame"/>
+        <child link="chassis"/>
+        <origin rpy="1.57 0.0 1.57" xyz="0.0 0.0 0.0" />
+    </joint>
     <link name="left_wheel">
       <inertial>
         <mass value="1.0"/>
-        <origin rpy="-0 -1e-06 3.14159" xyz="0.049227 0.011061 0.000747"/>
+        <origin rpy="0.0 0.0 0.0" xyz="0.0 0.0 0.0"/>
         <inertia
           ixx = "0.166667"
@@ -57,5 +70,5 @@
       <inertial>
         <mass value="1.0"/>
-        <origin rpy="0 0 0" xyz="-0.048887 0.00846 0.000728"/>
+        <origin rpy="0.0 0.0 0.0" xyz="0.0 0.0 0.0"/>
         <inertia
           ixx = "0.166667"
@@ -86,5 +99,5 @@
     </joint>
     <joint name='left_wheel_hinge' type='revolute'>
-      <origin rpy="0.0 0.0 0.0 " xyz="0.0 0.0 0.0"/>
+      <origin rpy="0.0 0.0 0.0 " xyz="-0.0497 0.00518 -0.03048"/>
       <child  link="left_wheel"/>
       <parent link="chassis"/>
@@ -93,5 +106,5 @@
     </joint>
     <joint name='right_wheel_hinge' type='revolute'>
-      <origin rpy="0.0 0.0 0.0 " xyz="0.0 0.0 0.0"/>
+      <origin rpy="0.0 3.14159 0.0 " xyz="0.0497 0.00518 -0.03048"/>
       <child  link="right_wheel"/>
       <parent link="chassis"/>

Commit message: Launch file (gazebo,joint states,spawn,bridge) and gazebo plugin

File: depthai_bridge/urdf/rae.urdf.xacro (robot description, xacro)
@@ -5,4 +5,6 @@
       <inertial>
         <mass value="1.0"/>
+        <mu1 value="0.001"/>
+        <mu2 value="0.001"/>
         <origin rpy="0.0 0.0 0.0" xyz="0.0 0.0 0.0"/>
         <inertia
@@ -93,9 +95,4 @@
       </visual>
     </link>
-    <joint name="base_joint" type="fixed">
-        <parent link="base_frame"/>
-        <child link="chassis"/>
-        <origin xyz="0 0 0" rpy="0 0 0" />
-    </joint>
     <joint name='left_wheel_hinge' type='revolute'>
       <origin rpy="0.0 0.0 0.0 " xyz="-0.0497 0.00518 -0.03048"/>
@@ -112,4 +109,17 @@
       <limit lower="-1e+16" upper="1e+16" effort="100" velocity="100"/>
     </joint>
+    <gazebo>
+        <plugin
+                filename="libignition-gazebo-diff-drive-system.so"
+                name="ignition::gazebo::systems::DiffDrive">
+                <left_joint>left_wheel_hinge</left_joint>
+                <right_joint>right_wheel_hinge</right_joint>
+                <wheel_separation>0.0994</wheel_separation>
+                <!-- check correct wheel radius when you come back to the task -->
+                <wheel_radius>0.0115</wheel_radius>
+                <odom_publish_frequency>1</odom_publish_frequency>
+                <topic>cmd_vel</topic>
+            </plugin>
+    </gazebo>
     <!-- <link name='body'>
       <inertial>
