Commit message: Adding caster wheels and improved mesh

File: depthai_bridge/urdf/inertial_moment_calc.xacro (robot description, xacro)
@@ -22,3 +22,12 @@
         </inertial>
     </xacro:macro>
+    <xacro:macro name="caster_wheels" params="mass r *origin">
+        <inertial>
+            <xacro:insert_block name="origin"/>
+            <mass value="${mass}" />
+            <inertia ixx="${(2/5) * mass * (r*r)}"  ixy="0.0" ixz="0.0"
+                    iyy="${(2/5) * mass * (r*r)}" iyz="0.0"
+                    izz="${(2/5) * mass * (r*r)}"/>
+        </inertial>
+    </xacro:macro>
 </robot>

File: depthai_bridge/urdf/rae.urdf.xacro (robot description, xacro)
@@ -1,24 +1,14 @@
 <?xml version="1.0"?>
 <robot name="rae" xmlns:xacro="http://ros.org/wiki/xacro">
+    <xacro:include filename="inertial_moment_calc.xacro"/>
     <link name="base_frame"/>
-    <link name="chassis">
-      <inertial>
-        <mass value="1.0"/>
-        <mu1 value="0.001"/>
-        <mu2 value="0.001"/>
-        <origin rpy="0.0 0.0 0.0" xyz="0.0 0.0 0.0"/>
-        <inertia
-          ixx = "0.166667"
-          ixy = "0"
-          ixz = "0"
-          iyy = "0.166667"
-          iyz = "0"
-          izz = "0.166667"
-        />
-      </inertial>
+<link name="chassis">
+      <xacro:body mass="0.2" d="0.125" h="0.028" w="0.1256">
+          <origin xyz="0 0.014 0.0" rpy="0.0 0.0 0.0"/>
+      </xacro:body>
       <collision>
         <origin rpy="0.0 0.0 0.0" xyz="0.0 0.0 0.0"/>
         <geometry>
-          <mesh filename="package://depthai_bridge/urdf/models/rae_chassis.stl" scale="1.0 1.0 1.0"/>
+          <mesh filename="package://depthai_bridge/urdf/models/RAE.stl" scale="1.0 1.0 1.0"/>
         </geometry>
       </collision>
@@ -26,9 +16,9 @@
         <origin rpy="0.0 0.0 0.0" xyz="0.0 0.0 0.0"/>
         <geometry>
-          <mesh filename="package://depthai_bridge/urdf/models/rae_chassis.stl" scale="1.0 1.0 1.0"/>
+          <mesh filename="package://depthai_bridge/urdf/models/RAE.stl" scale="1.0 1.0 1.0"/>
         </geometry>
         <material name="mat">
           <lighting>1</lighting>
-          <!-- <color rgba="0.1 0.1 0.1 1.0"/> -->
+          <color rgba="0.1 0.1 0.1 1.0"/>
           <shader type='pixel'/>
           <emissive>0 0 0 1</emissive>
@@ -41,105 +31,78 @@
         <parent link="base_frame"/>
         <child link="chassis"/>
-        <origin rpy="1.57 0.0 1.57" xyz="0.0 0.0 0.0" />
+        <origin rpy="1.57 0.0 1.57" xyz="0.0307 0.0 0.0" />
     </joint>
     <link name="left_wheel">
-      <inertial>
-        <mass value="1.0"/>
-        <origin rpy="0.0 0.0 0.0" xyz="0.0 0.0 0.0"/>
-        <inertia
-          ixx = "0.166667"
-          ixy = "0"
-          ixz = "0"
-          iyy = "0.166667"
-          iyz = "0"
-          izz = "0.166667"
-        />
-      </inertial>
+      <xacro:wheels mass="0.05" h="0.01" r="0.0125">
+            <origin xyz="-0.005 0.0 0.0" rpy="0.0 0.0 0.0"/>
+      </xacro:wheels>
+      <collision>
+        <origin rpy="0.0 0.0 0.0" xyz="-0.0125 0.0 0.0"/>
+        <geometry>
+            <mesh filename="package://depthai_bridge/urdf/models/Motor-wheel.stl" scale="1.0 1.0 1.0"/>
+        </geometry>
+      </collision>
+      <visual>
+        <origin rpy="0.0 0.0 0.0" xyz="-0.0125 0.0 0.0"/>
+        <geometry>
+            <mesh filename="package://depthai_bridge/urdf/models/Motor-wheel.stl" scale="1.0 1.0 1.0"/>
+        </geometry>
+      </visual>
+    </link>
+    <link name="right_wheel">
+      <xacro:wheels mass="0.05" h="0.01" r="0.0125">
+            <origin xyz="-0.005 0.0 0.0" rpy="0.0 0.0 0.0"/>
+      </xacro:wheels>
+      <collision>
+        <origin rpy="0.0 0.0 0.0" xyz="-0.0125 0.0 0.0"/>
+        <geometry>
+            <mesh filename="package://depthai_bridge/urdf/models/Motor-wheel.stl" scale="1.0 1.0 1.0"/>
+        </geometry>
+      </collision>
+      <visual>
+        <origin rpy="0.0 0.0 0.0" xyz="-0.0125 0.0 0.0"/>
+        <geometry>
+            <mesh filename="package://depthai_bridge/urdf/models/Motor-wheel.stl" scale="1.0 1.0 1.0"/>
+        </geometry>
+      </visual>
+    </link>
+    <joint name='left_wheel_hinge' type='continuous'>
+      <origin rpy="0.0 0.0 -1.57 " xyz="0.0 0.0427 0.0052"/>
+      <child  link="left_wheel"/>
+      <parent link="base_frame"/>
+      <axis rpy="0 0 0" xyz="-1 0 0"/>
+    </joint>
+    <joint name='right_wheel_hinge' type='continuous'>
+      <origin rpy="0.0 0.0 1.57 " xyz="0.0 -0.0427 0.0052"/>
+      <child  link="right_wheel"/>
+      <parent link="base_frame"/>
+      <axis rpy="0 0 0" xyz="1 0 0"/>
+    </joint>
+    <link name="left_caster_wheel">
+      <xacro:caster_wheels mass="0.05" r="0.005">
+            <origin xyz="0.0 0.0 0.0" rpy="0.0 0.0 0.0"/>
+      </xacro:caster_wheels>
       <collision>
         <origin rpy="0.0 0.0 0.0" xyz="0.0 0.0 0.0"/>
         <geometry>
-            <mesh filename="package://depthai_bridge/urdf/models/rae_wheel.stl" scale="1.0 1.0 1.0"/>
+          <mesh filename="package://depthai_bridge/urdf/models/caster-wheel.stl" scale="1.0 1.0 1.0"/>
         </geometry>
+        <surface>
+          <friction>
+            <ode>
+              <mu>0.01</mu>
+              <mu2>0.01</mu2>
+            </ode>
+          </friction>
+        </surface>
       </collision>
       <visual>
         <origin rpy="0.0 0.0 0.0" xyz="0.0 0.0 0.0"/>
         <geometry>
-            <mesh filename="package://depthai_bridge/urdf/models/rae_wheel.stl" scale="1.0 1.0 1.0"/>
+          <mesh filename="package://depthai_bridge/urdf/models/caster-wheel.stl" scale="1.0 1.0 1.0"/>
         </geometry>
-      </visual>
-    </link>
-    <link name="right_wheel">
-      <inertial>
-        <mass value="1.0"/>
-        <origin rpy="0.0 0.0 0.0" xyz="0.0 0.0 0.0"/>
-        <inertia
-          ixx = "0.166667"
-          ixy = "0"
-          ixz = "0"
-          iyy = "0.166667"
-          iyz = "0"
-          izz = "0.166667"
-        />
-      </inertial>
-      <collision>
-        <origin rpy="0.0 0.0 0.0" xyz="0.0 0.0 0.0"/>
-        <geometry>
-            <mesh filename="package://depthai_bridge/urdf/models/rae_wheel.stl" scale="1.0 1.0 1.0"/>
-        </geometry>
-      </collision>
-      <visual>
-        <origin rpy="0.0 0.0 0.0" xyz="0.0 0.0 0.0"/>
-        <geometry>
-            <mesh filename="package://depthai_bridge/urdf/models/rae_wheel.stl" scale="1.0 1.0 1.0"/>
-        </geometry>
-      </visual>
-    </link>
-    <joint name='left_wheel_hinge' type='revolute'>
-      <origin rpy="0.0 0.0 0.0 " xyz="-0.0497 0.00518 -0.03048"/>
-      <child  link="left_wheel"/>
-      <parent link="chassis"/>
-      <axis rpy="0 0 0" xyz="1 0 0"/>
-      <limit lower="-1e+16" upper="1e+16" effort="100" velocity="100"/>
-    </joint>
-    <joint name='right_wheel_hinge' type='revolute'>
-      <origin rpy="0.0 3.14159 0.0 " xyz="0.0497 0.00518 -0.03048"/>
-      <child  link="right_wheel"/>
-      <parent link="chassis"/>
-      <axis rpy="0 0 0" xyz="1 0 0"/>
-      <limit lower="-1e+16" upper="1e+16" effort="100" velocity="100"/>
-    </joint>
-    <gazebo>
-        <plugin
-                filename="libignition-gazebo-diff-drive-system.so"
-                name="ignition::gazebo::systems::DiffDrive">
-                <left_joint>left_wheel_hinge</left_joint>
-                <right_joint>right_wheel_hinge</right_joint>
-                <wheel_separation>0.0994</wheel_separation>
-                <!-- check correct wheel radius when you come back to the task -->
-                <wheel_radius>0.0115</wheel_radius>
-                <odom_publish_frequency>1</odom_publish_frequency>
-                <topic>cmd_vel</topic>
-            </plugin>
-    </gazebo>
-    <!-- <link name='body'>
-      <inertial>
-        <mass value="1.0"/>
-        <inertia
-          ixx ="0.166667"
-          ixy = "0"
-          ixz = "0"
-          iyy = "0.166667"
-          iyz = "0"
-          izz = "0.166667"
-        />
-      </inertial>
-      <visual>
-        <pose>0 0 0 0 -0 0</pose>
-        <geometry>
-          <mesh filename = "/home/sags/Downloads/RAE-ASSY-1006.stl"/>
-        </geometry>
-        <material>
+        <material name="mat">
           <lighting>1</lighting>
-            <color rgba="0.8 0.8 0.8 0.8"/>
+          <color rgba="1.0 1.0 1.0 1.0"/>
           <shader type='pixel'/>
           <emissive>0 0 0 1</emissive>
@@ -148,60 +111,47 @@
         <cast_shadows>1</cast_shadows>
       </visual>
-      <collision name='collision'>
-        <laser_retro>0</laser_retro>
-        <max_contacts>10</max_contacts>
-        <pose>0 0 0 0 -0 0</pose>
+    </link>
+    <joint name="base_left_caster_wheel" type="fixed">
+        <parent link="base_frame"/>
+        <child link="left_caster_wheel"/>
+        <origin rpy="0.0 0.0 0.0" xyz="0.0735 0.0445 -0.001" />
+    </joint>
+    <link name="right_caster_wheel">
+      <xacro:caster_wheels mass="0.05" r="0.005">
+            <origin xyz="0.0 0.0 0.0" rpy="0.0 0.0 0.0"/>
+      </xacro:caster_wheels>
+      <collision>
+        <origin rpy="0.0 0.0 0.0" xyz="0.0 0.0 0.0"/>
         <geometry>
-          <mesh>
-            <uri>/home/sags/Downloads/RAE-ASSY-1006.stl</uri>
-            <scale>1 1 1</scale>
-          </mesh>
+          <mesh filename="package://depthai_bridge/urdf/models/caster-wheel.stl" scale="1.0 1.0 1.0"/>
         </geometry>
         <surface>
           <friction>
             <ode>
-              <mu>1</mu>
-              <mu2>1</mu2>
-              <fdir1>0 0 0</fdir1>
-              <slip1>0</slip1>
-              <slip2>0</slip2>
+              <mu>0.01</mu>
+              <mu2>0.01</mu2>
             </ode>
-            <torsional>
-              <coefficient>1</coefficient>
-              <patch_radius>0</patch_radius>
-              <surface_radius>0</surface_radius>
-              <use_patch_radius>1</use_patch_radius>
-              <ode>
-                <slip>0</slip>
-              </ode>
-            </torsional>
           </friction>
-          <bounce>
-            <restitution_coefficient>0</restitution_coefficient>
-            <threshold>1e+06</threshold>
-          </bounce>
-          <contact>
-            <collide_without_contact>0</collide_without_contact>
-            <collide_without_contact_bitmask>1</collide_without_contact_bitmask>
-            <collide_bitmask>1</collide_bitmask>
-            <ode>
-              <soft_cfm>0</soft_cfm>
-              <soft_erp>0.2</soft_erp>
-              <kp>1e+13</kp>
-              <kd>1</kd>
-              <max_vel>0.01</max_vel>
-              <min_depth>0</min_depth>
-            </ode>
-            <bullet>
-              <split_impulse>1</split_impulse>
-              <split_impulse_penetration_threshold>-0.01</split_impulse_penetration_threshold>
-              <soft_cfm>0</soft_cfm>
-              <soft_erp>0.2</soft_erp>
-              <kp>1e+13</kp>
-              <kd>1</kd>
-            </bullet>
-          </contact>
         </surface>
       </collision>
-    </link> -->
+      <visual>
+        <origin rpy="0.0 0.0 0.0" xyz="0.0 0.0 0.0"/>
+        <geometry>
+          <mesh filename="package://depthai_bridge/urdf/models/caster-wheel.stl" scale="1.0 1.0 1.0"/>
+        </geometry>
+        <material name="mat">
+          <lighting>1</lighting>
+          <color rgba="1.0 1.0 1.0 1.0"/>
+          <shader type='pixel'/>
+          <emissive>0 0 0 1</emissive>
+        </material>
+        <transparency>0</transparency>
+        <cast_shadows>1</cast_shadows>
+      </visual>
+    </link>
+    <joint name="base_right_caster_wheel" type="fixed">
+        <parent link="base_frame"/>
+        <child link="right_caster_wheel"/>
+        <origin rpy="0.0 0.0 0.0" xyz="0.0735 -0.0445 -0.001" />
+    </joint>
 </robot>

File: depthai_bridge/urdf/rae_gazebo.urdf.xacro (robot description, xacro)
@@ -4,5 +4,5 @@
     <link name="base_frame"/>
     <link name="chassis">
-      <xacro:body mass="0.2" d="0.125" h="0.028" w="0.1256">
+      <xacro:body mass="0.5" d="0.125" h="0.028" w="0.1256">
           <origin xyz="0 0.014 0.0" rpy="0.0 0.0 0.0"/>
       </xacro:body>
@@ -12,12 +12,4 @@
           <mesh filename="package://depthai_bridge/urdf/models/RAE-enclosure_01051900.stl" scale="0.001 0.001 0.001"/>
         </geometry>
-        <surface>
-          <friction>
-            <ode>
-              <mu>0.01</mu>
-              <mu2>0.01</mu2>
-            </ode>
-          </friction>
-        </surface>
       </collision>
       <visual>
@@ -36,9 +28,4 @@
       </visual>
     </link>
-    <gazebo reference="chassis">
-       <material>Gazebo/Black</material>
-        <mu1>0.001</mu1>
-        <mu2>0.001</mu2>
-    </gazebo>
     <joint name="base_chassis_joint" type="fixed">
         <parent link="base_frame"/>
@@ -92,4 +79,80 @@
       <axis rpy="0 0 0" xyz="1 0 0"/>
     </joint>
+    <link name="left_caster_wheel">
+      <xacro:caster_wheels mass="0.035" r="0.005">
+            <origin xyz="0.0 0.0 0.0" rpy="0.0 0.0 0.0"/>
+      </xacro:caster_wheels>
+      <collision>
+        <origin rpy="0.0 0.0 0.0" xyz="0.0 0.0 0.0"/>
+        <geometry>
+          <mesh filename="package://depthai_bridge/urdf/models/caster-wheel.stl" scale="1.0 1.0 1.0"/>
+        </geometry>
+        <surface>
+          <friction>
+            <ode>
+              <mu>0.01</mu>
+              <mu2>0.01</mu2>
+            </ode>
+          </friction>
+        </surface>
+      </collision>
+      <visual>
+        <origin rpy="0.0 0.0 0.0" xyz="0.0 0.0 0.0"/>
+        <geometry>
+          <mesh filename="package://depthai_bridge/urdf/models/caster-wheel.stl" scale="1.0 1.0 1.0"/>
+        </geometry>
+        <material name="mat">
+          <lighting>1</lighting>
+          <color rgba="1.0 1.0 1.0 1.0"/>
+          <shader type='pixel'/>
+          <emissive>0 0 0 1</emissive>
+        </material>
+        <transparency>0</transparency>
+        <cast_shadows>1</cast_shadows>
+      </visual>
+    </link>
+    <joint name="base_left_caster_wheel" type="fixed">
+        <parent link="base_frame"/>
+        <child link="left_caster_wheel"/>
+        <origin rpy="0.0 0.0 0.0" xyz="0.0735 0.0445 -0.001" />
+    </joint>
+    <link name="right_caster_wheel">
+      <xacro:caster_wheels mass="0.035" r="0.005">
+            <origin xyz="0.0 0.0 0.0" rpy="0.0 0.0 0.0"/>
+      </xacro:caster_wheels>
+      <collision>
+        <origin rpy="0.0 0.0 0.0" xyz="0.0 0.0 0.0"/>
+        <geometry>
+          <mesh filename="package://depthai_bridge/urdf/models/caster-wheel.stl" scale="1.0 1.0 1.0"/>
+        </geometry>
+        <surface>
+          <friction>
+            <ode>
+              <mu>0.01</mu>
+              <mu2>0.01</mu2>
+            </ode>
+          </friction>
+        </surface>
+      </collision>
+      <visual>
+        <origin rpy="0.0 0.0 0.0" xyz="0.0 0.0 0.0"/>
+        <geometry>
+          <mesh filename="package://depthai_bridge/urdf/models/caster-wheel.stl" scale="1.0 1.0 1.0"/>
+        </geometry>
+        <material name="mat">
+          <lighting>1</lighting>
+          <color rgba="1.0 1.0 1.0 1.0"/>
+          <shader type='pixel'/>
+          <emissive>0 0 0 1</emissive>
+        </material>
+        <transparency>0</transparency>
+        <cast_shadows>1</cast_shadows>
+      </visual>
+    </link>
+    <joint name="base_right_caster_wheel" type="fixed">
+        <parent link="base_frame"/>
+        <child link="right_caster_wheel"/>
+        <origin rpy="0.0 0.0 0.0" xyz="0.0735 -0.0445 -0.001" />
+    </joint>
     <gazebo>
         <plugin
